File: KiCad/Power_USB.kicad_sch (KiCad schematic)
At the start: 11 parts, among them U1 AP2112K-3.3, U2 TLV70218DBVR

Commit message: final cleanups and other fixes
Parts:
- D1: value 1n4002W -> 1n5819W
Changed lines of the file:
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@@
 			)
 		)
-		(property "Value" "1n4002W"
+		(property "Value" "1n5819W"
 			(at 66.04 33.6296 0)
 			(effects

Commit message: updated part values, generated production files
Other:
- note added: "D1 NEEDS to be 0omh resistor or schottky"
- note removed: "D1 NEEDS to be 0omh resistor or 1n4002"
- note removed: "KoreanHROParts USB_C_Receptacle_HRO_TYPE-C-31-M-12"
Changed lines of the file:
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@@
-		)
-	)
-	(text "KoreanHROParts \nUSB_C_Receptacle_HRO_TYPE-C-31-M-12"
-		(exclude_from_sim no)
-		(at 38.735 57.785 0)
-		(effects
-			(font
-				(size 1.27 1.27)
-			)
-			(justify left bottom)
 		)
 	)
@@
 		)
 	)
-	(text "D1 NEEDS to be 0omh resistor or 1n4002"
+	(text "D1 NEEDS to be 0omh resistor or schottky"
 		(exclude_from_sim no)
-		(at 50.8 29.21 0)
+		(at 49.53 40.64 0)
 		(effects
 			(font
